File: MIKROE_MODBUS/MODBUS_CLIX/MODBUS_CLIX.kicad_pcb (KiCad board)
At the start: 2 copper layers, 25.4 x 53.6 mm, 40 parts, among them J1 Conn_01x02_Pin, J10 Conn_01x02_Pin, J11 Conn_01x03_Pin, J12 Conn_01x02_Pin, J2 Conn_01x02_Pin, J3 Conn_01x02_Pin, J4 Conn_01x02_Pin, J5 Conn_01x02_Pin, J6 Conn_01x02_Pin, J7 TERMINAL BLOCK, J8 Conn_01x02_Pin, J9 Conn_01x02_Pin, U1 CLICK BOARD, U2 MAX485E, U3 MT3608

Commit message: -
Parts:
- removed J1, J2, J3, J5, J9: Conn_01x02_Pin, Connector_PinHeader_2.54mm:PinHeader_1x02_P2.54mm_Vertical
- removed R11: 14.3K, Resistor_SMD:R_0603_1608Metric_Pad0.98x0.95mm_HandSolder
- removed R8: 75K, Resistor_SMD:R_0603_1608Metric_Pad0.98x0.95mm_HandSolder
- removed R9: 10K, Resistor_SMD:R_0603_1608Metric_Pad0.98x0.95mm_HandSolder
- added JP1: SolderJumper_2_Open, Jumper:SolderJumper-2_P1.3mm_Open_Pad1.0x1.5mm, F.Cu at (168.5, 62.0)
- added JP2: SolderJumper_2_Open, Jumper:SolderJumper-2_P1.3mm_Open_Pad1.0x1.5mm, F.Cu at (168.5, 53.1)
- added JP4: SolderJumper_3_Open, Jumper:SolderJumper-3_P1.3mm_Open_Pad1.0x1.5mm, F.Cu at (159.6, 92.2)
- added kibuzzard-67110E36: G***, kibuzzard-67110E36, F.Cu at (178.6, 51.8)
- added kibuzzard-67110F70: G***, kibuzzard-67110F70, F.Cu at (178.3, 59.1)
- added kibuzzard-67110FB4: G***, kibuzzard-67110FB4, F.Cu at (178.3, 64.7)
- R10: value 270k -> 91K
- R12: value 69.8K -> 180K
- R13: value 1.8K -> 4.7K
- moved G*** 30.4 mm to (152.3, 44.4), turned to -30 degrees
- moved R14 12.9 mm to (168.5, 55.4)
- moved RV1 12.6 mm to (172.1, 47.9)
- moved R12 8.76 mm to (168.5, 59.1), turned to 180 degrees
- moved J4 8.66 mm to (172.6, 64.7), turned to 90 degrees
- moved J7 7.62 mm to (163.3, 92.0), turned to 0 degrees
- moved J10 6.61 mm to (172.6, 54.1), turned to 90 degrees
- moved D1 6.36 mm to (162.6, 64.7)
- moved R13 6.34 mm to (172.0, 61.9), turned to 0 degrees
- moved J6 5.60 mm to (172.6, 59.1), turned to 90 degrees
- moved R10 5.23 mm to (168.5, 64.7), turned to 180 degrees
- moved R7 3.08 mm to (161.9, 49.0)
- moved C3 2.91 mm to (157.3, 52.6)
- moved C4 2.91 mm to (158.8, 52.1)
- moved U3 2.91 mm to (161.8, 51.7)
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Connections:
- J7 pad 1: GNDD -> V_SLAVE
- J7 pad 2: MASTER_MODBUS_B -> MASTER_MODBUS_A
- J7 pad 3: MASTER_MODBUS_A -> MASTER_MODBUS_B
- J7 pad 4: +VOUT -> GNDD
- J8 pad 1: +VOUT -> V_SLAVE
- R10 pad 2: Net-(J3-Pin_1) -> Net-(JP1-B)
- R12 pad 2: Net-(J5-Pin_1) -> Net-(JP1-B)
- R13 pad 1: Net-(J5-Pin_1) -> Net-(JP1-B)
Routing:
- net V_SLAVE: track 0.00 -> 31.7 mm
- net +5V_MIKROE: track 67.7 -> 88.1 mm, vias 0 -> 2
- net +VOUT: track 67.1 -> 49.7 mm
- net Net-(J1-Pin_1): track 16.8 -> 0.00 mm
- net Net-(J3-Pin_1): track 16.7 -> 0.00 mm
- net Net-(J5-Pin_1): track 16.2 -> 0.00 mm
- net Net-(J2-Pin_2): track 11.8 -> 0.00 mm
- net Net-(D1-A): track 11.0 -> 21.1 mm
- net Net-(JP1-B): track 0.00 -> 8.83 mm
- net Net-(R14-Pad1): track 3.58 -> 8.93 mm, vias 0 -> 2
- net Net-(J4-Pin_2): track 11.1 -> 7.50 mm
- net Net-(J6-Pin_2): track 10.3 -> 7.46 mm
- net /GPIO1: track 15.2 -> 17.5 mm
- net GNDD: track 8.34 -> 10.5 mm, vias 12 -> 16
- net Net-(J10-Pin_2): track 8.52 -> 6.39 mm
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- removed copper zone on F.Cu, net Net-(D1-A)
Other:
- board size 25.4 x 53.6 mm -> 25.4 x 52.6 mm
- board text added: "EN"
- board text added: "VO"
- board text removed: "12V"
- board text removed: "24V"
- board text removed: "POT"
