File: MIKROE_MODBUS/MODBUS_CLIX/MODBUS_CLIX.kicad_pcb (KiCad board)
At the start: 2 copper layers, 25.4 x 52.6 mm, 38 parts, among them J10 Conn_01x02_Pin, J11 Conn_01x03_Pin, J12 Conn_01x02_Pin, J4 Conn_01x02_Pin, J6 Conn_01x02_Pin, J7 TERMINAL BLOCK, J8 Conn_01x02_Pin, U1 CLICK BOARD, U2 MAX485E, U3 MT3608

Commit message: Initial Design Review
1. Set unused MikroE pins to Unconnected
2. Edited Silk Screen details
Parts:
- moved G*** 3.55 mm to (151.1, 47.7), turned to 0 degrees
Connections:
- U1 pad 11: /SDA -> unconnected-(U1-SDA-Pad11)
- U1 pad 12: /SCL -> unconnected-(U1-SCL-Pad12)
- U1 pad 2: /RST -> unconnected-(U1-RST-Pad2)
- U1 pad 3: /CS -> unconnected-(U1-CS-Pad3)
- U1 pad 4: /SCK -> unconnected-(U1-SCK-Pad4)
- U1 pad 5: /MISO -> unconnected-(U1-MISO-Pad5)
- U1 pad 6: /MOSI -> unconnected-(U1-MOSI-Pad6)
- U1 pad 7: /3.3V -> unconnected-(U1-+3.3V-Pad7)
Other:
- board text added: "BST"
- board text added: "DI"
- board text added: "G"
- board text added: "POW"
- board text added: "RO"
- board text removed: "PWR"
- board text removed: "RX"
- board text removed: "TX"

Commit message: -
Parts:
- removed kibuzzard-67110E36: G***, kibuzzard-67110E36
- added JP5: SolderJumper_2_Open, Jumper:SolderJumper-2_P1.3mm_Open_Pad1.0x1.5mm, B.Cu at (170.8, 87.0)
- added kibuzzard-6715C691: G***, kibuzzard-6715C691, F.Cu at (178.6, 51.8)
- added kibuzzard-6715C801: G***, kibuzzard-6715C801, F.Cu at (160.3, 69.6)
- added kibuzzard-6715C814: G***, kibuzzard-6715C814, F.Cu at (160.3, 72.3)
- added kibuzzard-6715C87B: G***, kibuzzard-6715C87B, F.Cu at (175.0, 69.6)
- added kibuzzard-6715C8B5: G***, kibuzzard-6715C8B5, F.Cu at (175.0, 72.3)
- added kibuzzard-6715C9CA: G***, kibuzzard-6715C9CA, F.Cu at (156.5, 57.1)
- added kibuzzard-6715CA09: G***, kibuzzard-6715CA09, F.Cu at (159.6, 89.2)
- added kibuzzard-6715CA18: G***, kibuzzard-6715CA18, F.Cu at (159.6, 95.2)
- added kibuzzard-6715CB0C: G***, kibuzzard-6715CB0C, F.Cu at (163.3, 96.6)
- added kibuzzard-6715CB35: G***, kibuzzard-6715CB35, F.Cu at (165.9, 96.6)
- added kibuzzard-6715CB51: G***, kibuzzard-6715CB51, F.Cu at (168.3, 96.7)
- added kibuzzard-6715CBD0: G***, kibuzzard-6715CBD0, F.Cu at (171.0, 96.7)
- added kibuzzard-6715CD4A: G***, kibuzzard-6715CD4A, F.Cu at (158.2, 76.3)
- added kibuzzard-6715CD61: G***, kibuzzard-6715CD61, F.Cu at (157.5, 94.0)
- added kibuzzard-6715CEA4: G***, kibuzzard-6715CEA4, F.Cu at (173.1, 93.7)
- added kibuzzard-6715CEBB: G***, kibuzzard-6715CEBB, F.Cu at (176.7, 91.3)
- added kibuzzard-6715CECC: G***, kibuzzard-6715CECC, F.Cu at (177.0, 94.0)
- added kibuzzard-6715CED3: G***, kibuzzard-6715CED3, F.Cu at (176.7, 83.9)
- added kibuzzard-6715CED8: G***, kibuzzard-6715CED8, F.Cu at (176.7, 81.5)
- added kibuzzard-6715CEDE: G***, kibuzzard-6715CEDE, F.Cu at (176.3, 76.3)
- added kibuzzard-6715CF5F: G***, kibuzzard-6715CF5F, F.Cu at (158.3, 59.7)
- added kibuzzard-6715CF9A: G***, kibuzzard-6715CF9A, F.Cu at (158.3, 64.7)
- added kibuzzard-6715CFC1: G***, kibuzzard-6715CFC1, F.Cu at (168.6, 51.3)
- added kibuzzard-6715CFD6: G***, kibuzzard-6715CFD6, F.Cu at (168.6, 60.3)
- added kibuzzard-6715D06D: G***, kibuzzard-6715D06D, B.Cu at (178.4, 63.8)
- added kibuzzard-6715D3D8: G***, kibuzzard-6715D3D8, B.Cu at (173.8, 86.9)
Connections:
- R6 pad 2: MASTER_MODBUS_B -> Net-(JP5-A)
Routing:
- net MASTER_MODBUS_B: track 40.0 -> 43.5 mm, vias 0 -> 1
- net Net-(JP5-A): track 0.00 -> 2.18 mm, vias 0 -> 1
Other:
- board text removed: "5V"
- board text removed: "A"
- board text removed: "B"
- board text removed: "BST"
- board text removed: "CTRL"
- board text removed: "DI"
- board text removed: "EN"
- board text removed: "G"
- board text removed: "GND"
- board text removed: "IO1"
- board text removed: "POW"
- board text removed: "R/T"
- board text removed: "RO"
- board text removed: "VCC"
- board text removed: "VO"

Commit message: -
panelization
Parts:
- removed kibuzzard-6715CFC1: G***, kibuzzard-6715CFC1
- removed kibuzzard-6715CFD6: G***, kibuzzard-6715CFD6
- added kibuzzard-671645B5: G***, kibuzzard-671645B5, F.Cu at (169.3, 52.5)
- added kibuzzard-671645C1: G***, kibuzzard-671645C1, F.Cu at (169.2, 60.5)
- U1: footprint MIKROE:MIKROE-PINS -> MIKROE_3800:MIKROE-3800
- moved U1 13.5 mm to (155.6, 94.0)
- moved G*** 1.85 mm to (150.2, 49.4)
- moved RV1 1.77 mm to (172.0, 49.7)
- moved kibuzzard-6715C691 1.15 mm to (178.3, 52.9)
- moved JP2 0.85 mm to (168.5, 54.0)
- moved R14 0.66 mm to (168.6, 56.0)
- moved J10 0.64 mm to (172.6, 54.8)
- moved kibuzzard-6715CB0C 0.21 mm to (163.3, 96.4)
- moved kibuzzard-6715CB35 0.21 mm to (166.0, 96.4)
- moved kibuzzard-6715CB51 0.21 mm to (168.3, 96.5)
- moved kibuzzard-6715CBD0 0.21 mm to (171.0, 96.5)
Routing:
- net GNDD: track 10.5 -> 13.3 mm, vias 16 -> 47
- net Net-(R14-Pad1): track 8.93 -> 7.35 mm
- net Net-(JP2-B): track 7.20 -> 5.80 mm
- net Net-(J10-Pin_2): track 6.39 -> 5.30 mm
- net +VOUT: track 49.7 -> 49.0 mm
- net /FB_PIN: track 19.3 -> 19.9 mm
- net GNDPWR: track 7.49 -> 7.74 mm, vias 14 -> 19
Other:
- board size 25.4 x 52.6 mm -> 25.4 x 50 mm
