File: MIKROE_RELAY/MIKROE_RELAY/_autosave-MIKROE_RELAY.kicad_pcb (KiCad board)
At the start: 2 copper layers, 32.7 x 53.5 mm, 24 parts, among them J1 RELAY1, J2 RELAY2, J3 Screw_Terminal_01x04, K1 SRD-05VDC-SL-C, K2 SRD-05VDC-SL-C, Q1 Q_NMOS_Depletion_GSD, Q2 Q_NMOS_Depletion_GSD, U2 B0505S-2WR3, U3 PC817, U4 PC817

Commit message: -
Parts:
- moved R3 73.5 mm to (124.2, 56.8)
- moved R2 72.9 mm to (107.8, 69.2), turned to -90 degrees
- moved D1 72.9 mm to (107.8, 72.8), turned to 90 degrees
- moved D2 71.5 mm to (122.2, 60.5)
- moved Q1 66.4 mm to (121.7, 57.2), turned to -90 degrees
- moved Q2 41.6 mm to (127.9, 57.2), turned to -90 degrees
- moved D4 37.9 mm to (127.4, 60.5), turned to 0 degrees
- moved D3 31.0 mm to (142.4, 72.7), turned to 90 degrees
- moved R8 30.3 mm to (131.4, 55.1), turned to 0 degrees
- moved R7 26.6 mm to (142.4, 69.2), turned to -90 degrees
- moved C1 5.34 mm to (139.5, 51.6), turned to -90 degrees
- moved C4 3.25 mm to (113.7, 51.7), turned to -90 degrees
- moved R1 2.21 mm to (107.3, 58.7)
- moved U3 2.21 mm to (114.0, 58.6)
- moved U4 2.08 mm to (135.6, 58.6)
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Other:
- board size 32.7 x 53.5 mm -> 37.8 x 53.5 mm
